Commit message: Some changes to improve training time

File: assets/urdfs/dynamic_titan.urdf (robot description, URDF)
Before this commit: robot titan, 69 links, 68 joints
Links:
- link left_10_wheel: mass 2.0 -> 2.637
- link left_11_wheel: mass 2.0 -> 2.637
- link left_1_wheel: mass 2.0 -> 2.637
- link left_2_wheel: mass 2.0 -> 2.637
- link left_3_wheel: mass 2.0 -> 2.637
- link left_4_wheel: mass 2.0 -> 2.637
- link left_5_wheel: mass 2.0 -> 2.637
- link left_6_wheel: mass 2.0 -> 2.637
- link left_7_wheel: mass 2.0 -> 2.637
- link left_8_wheel: mass 2.0 -> 2.637
- link left_9_wheel: mass 2.0 -> 2.637
- link right_10_wheel: mass 2.0 -> 2.637
- link right_11_wheel: mass 2.0 -> 2.637
- link right_1_wheel: mass 2.0 -> 2.637
- link right_2_wheel: mass 2.0 -> 2.637
- link right_3_wheel: mass 2.0 -> 2.637
- link right_4_wheel: mass 2.0 -> 2.637
- link right_5_wheel: mass 2.0 -> 2.637
- link right_6_wheel: mass 2.0 -> 2.637
- link right_7_wheel: mass 2.0 -> 2.637
- link right_8_wheel: mass 2.0 -> 2.637
- link right_9_wheel: mass 2.0 -> 2.637
