Commit message: Expert Function Including Corner Distances

File: Wall_URDF/Wall.urdf (robot description, URDF)
Before this commit: robot block_2, 1 links, 0 joints
Links:
- link block_2_base_link: geometry collision box size=.5 22 1; visual box size=.5 22 1

File: Wall_URDF/Wall2.urdf (robot description, URDF)
Before this commit: robot block_2, 1 links, 0 joints
Links:
- link block_2_base_link: geometry collision box size=22 .5 1; visual box size=22 .5 1
